File: KiCad Files/TLV320ADC6120/TLV320ADC6120_Board.kicad_pcb (KiCad board)
At the start: 2 copper layers, 27.9 x 48.3 mm, 33 parts, among them J1 Conn_01x10, J2 Conn_01x10, J3 AudioJack3, J4 Conn_01x02, J5 Conn_01x02, U1 TPS7A0533PDBV, U2 TPS7A0533PDBV

Commit message: Fix part number
TLV320ADC6120 mistakenly labelled as a second TPS7A0533PDBV
Parts:
- U2: value TPS7A0533PDBV -> TLV320ADC6120
Changed lines of the file:
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@@
       (effects (font (size 1 1) (thickness 0.15)))
     )
-    (fp_text value "TPS7A0533PDBV" (at 0 3.05 90) (layer "F.Fab")
+    (fp_text value "TLV320ADC6120" (at 0 3.05 90) (layer "F.Fab")
       (effects (font (size 1 1) (thickness 0.15)))
     )

Commit message: Fix part number
Changed mislabeled
TPS7A0533PDBV to TPS7A2031PDBVR on the TLV320ADC6120 board
Parts:
- U1: value TPS7A0533PDBV -> TPS7A2031PDBVR
Changed lines of the file:
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@@
       (effects (font (size 1 1) (thickness 0.15)))
     )
-    (fp_text value "TPS7A0533PDBV" (at 0 2.4 90) (layer "F.Fab")
+    (fp_text value "TPS7A2031PDBVR" (at 0 2.4 90) (layer "F.Fab")
       (effects (font (size 1 1) (thickness 0.15)))
     )
