File: KiCad Files/TLV320ADC6120/TLV320ADC6120_Board.kicad_sch (KiCad schematic)
At the start: 33 parts, among them J1 Conn_01x10, J2 Conn_01x10, J3 AudioJack3, J4 Conn_01x02, J5 Conn_01x02, U1 TPS7A0533PDBV, U2 TPS7A0533PDBV

Commit message: Fix part number
TLV320ADC6120 mistakenly labelled as a second TPS7A0533PDBV
Parts:
- U2: value TPS7A0533PDBV -> TLV320ADC6120
Changed lines of the file:
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@@
     (in_bom yes) (on_board yes) (fields_autoplaced)
     (property "Reference" "U2" (id 0) (at 180.34 53.34 0))
-    (property "Value" "TPS7A0533PDBV" (id 1) (at 180.34 55.88 0))
+    (property "Value" "TLV320ADC6120" (id 1) (at 180.34 55.88 0))
     (property "Footprint" "Library:QFN-16_EP_3x3_Pitch0.5mm" (id 2) (at 180.34 104.14 0)
       (effects (font (size 1.27 1.27)) hide)
@@
     )
     (path "/3076b0f6-3b15-4eee-861e-b6955be460f2"
-      (reference "U2") (unit 1) (value "TPS7A0533PDBV") (footprint "Library:QFN-16_EP_3x3_Pitch0.5mm")
-    )
-  )
+      (reference "U2") (unit 1) (value "TLV320ADC6120") (footprint "Library:QFN-16_EP_3x3_Pitch0.5mm")
+    )
+  )

Commit message: Fix part number
Changed mislabeled
TPS7A0533PDBV to TPS7A2031PDBVR on the TLV320ADC6120 board
Parts:
- U1: value TPS7A0533PDBV -> TPS7A2031PDBVR
Changed lines of the file:
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@@
     (in_bom yes) (on_board yes) (fields_autoplaced)
     (property "Reference" "U1" (id 0) (at 58.42 38.1 0))
-    (property "Value" "TPS7A0533PDBV" (id 1) (at 58.42 40.64 0))
+    (property "Value" "TPS7A2031PDBVR" (id 1) (at 58.42 40.64 0))
     (property "Footprint" "Package_TO_SOT_SMD:SOT-23-5" (id 2) (at 58.42 39.37 0)
       (effects (font (size 1.27 1.27)) hide)
@@
     )
     (path "/63d014fd-19cc-4a1b-822f-c2950ee2f950"
-      (reference "U1") (unit 1) (value "TPS7A0533PDBV") (footprint "Package_TO_SOT_SMD:SOT-23-5")
+      (reference "U1") (unit 1) (value "TPS7A2031PDBVR") (footprint "Package_TO_SOT_SMD:SOT-23-5")
     )
     (path "/3076b0f6-3b15-4eee-861e-b6955be460f2"
