File: Plug-in Sub-Boards/LCD-1.9in-GUI/Schematics/stm32.kicad_sch (KiCad schematic)
At the start: 32 parts, among them J201 Conn_ST_STDC14, SW302 SW_Push, SW303 SW_Push, SW304 SW_Push, U202 W25Q16, U301 STM32G431CBUx, Y301 8MHz

Commit message: Cleanup
Parts:
- removed C304 (x2), C306: 100nF, Capacitor_SMD:C_0402_1005Metric, symbol Device:C
- removed C306: 4.7uF, Capacitor_SMD:C_0603_1608Metric, symbol Device:C
- removed R306 (x2): 100k, Resistor_SMD:R_0402_1005Metric, symbol Device:R
- removed R306: 2k, Resistor_SMD:R_0402_1005Metric, symbol Device:R
- added C304 (x2), C306: 100nF, Capacitor_SMD:C_0402_1005Metric, symbol Device:C
- added C306: 4.7uF, Capacitor_SMD:C_0603_1608Metric, symbol Device:C
- added R306 (x2): 100k, Resistor_SMD:R_0402_1005Metric, symbol Device:R
- added R306: 2k, Resistor_SMD:R_0402_1005Metric, symbol Device:R
Connections:
- net +3.3V: now also C304.1, C304.1, R306.1, R306.1
- net GND: now also C304.2, C304.2, C306.2, C306.2, R306.2
- net SPI_MISO: now also R306.1
- net SPI_NSS: now also R306.2
- net VDDA: now also C306.1, C306.1
- net at D301.2 (K1): now also R306.2
- net CARD_DETECT_0: no longer names the net of U301.25 (PB12)
- net CARD_DETECT_1: no longer names the net of U301.26 (PB13)
- net SAI-A-FS: no longer names the net of U301.31 (PA9)
- net SAI-A-GPIO0: no longer names the net of U301.29 (PC6)
- net SAI-A-GPIO1: no longer names the net of U301.28 (PB15)
- net SAI-A-MCLK: no longer names the net of U301.11 (PA3)
- net SAI-A-SCK: no longer names the net of U301.30 (PA8)
- net SAI-A-SD: no longer names the net of U301.32 (PA10)
- net SAI-B-FS: no longer names the net of U301.44 (PB6)
- net SAI-B-GPIO0: no longer names the net of U301.39 (PC10)
- net SAI-B-GPIO1: no longer names the net of U301.40 (PC11)
- net SAI-B-MCLK: no longer names the net of U301.42 (PB4)
- net SAI-B-SCK: no longer names the net of U301.41 (PB3)
- net SAI-B-SD: no longer names the net of U301.43 (PB5)
Other:
- note added: "Reset Button"
- title: STM32 USB Audio Interface - STM32G431 -> (none)
