File: STM32-USB-Audio-Board/STM32-USB-Audio-Board.kicad_sch (KiCad schematic)
At the start: 0 parts

Commit message: Cleanup
Parts:
- added H101, H102, H103, H104, H105: MountingHole_Pad, MountingHole:MountingHole_2.2mm_M2_Pad_Via, symbol Mechanical:MountingHole_Pad
Connections:
- new net GND: H101.1, H102.1, H103.1, H104.1, H105.1
Other:
- sheet DAPLink CH32V305 renamed DAPLink CH32V203
- sheet USB Connector and Power Supply renamed USB Connector
- removed sheet Display and Buttons
- added sheet HMI Sub-board Connector (Schematics/conn_hmi.kicad_sch)
- added sheet Power Supply (Schematics/pwr.kicad_sch)
- sheet DAPLink CH32V203: file Schematics/mcu_daplink_ch32v305.kicad_sch -> Schematics/mcu_daplink_ch32v203.kicad_sch
- sheet DAPLink CH32V203 ports: added USB_DN, USB_DP; removed USB_HS_DN, USB_HS_DP
- sheet STM32G431CBU6 ports: added USART3_RX, USART3_TX; removed ENC_A, ENC_B, ENC_BTN, LCD_BLK, LCD_DC, LCD_RES, LCD_SPI_MISO, LCD_SPI_MOSI, LCD_SPI_NSS, LCD_SPI_SCK
- sheet USB Connector: file conn_usb_pwr.kicad_sch -> Schematics/conn_usb.kicad_sch
- note added: "HP/SPK"
- note added: "Mic"
