File: STM32-USB-Audio-Board/Schematics/conn_usb.kicad_sch (KiCad schematic)
At the start: 37 parts, among them J301 USB_C_Receptacle_USB2.0, U301 FE1.1s, U302 USBLC6-2SC6, U803 SY8883DFC, Y301 12MHz

Commit message: Cleanup
Parts:
- removed C206: 10uF, Capacitor_Tantalum_SMD:CP_EIA-3528-21_Kemet-B, symbol Device:C_Polarized
- removed C801: 10pF, Capacitor_SMD:C_0402_1005Metric, symbol Device:C
- removed C802: 4.7uF, Capacitor_SMD:C_0603_1608Metric, symbol Device:C
- removed C804: 10uF, Capacitor_SMD:C_0603_1608Metric, symbol Device:C
- removed L302: L_Ferrite_Coupled, symbol Device:L_Ferrite_Coupled
- removed L801: 1uH, Inductor_SMD:L_Sunlord_SWPA4020S, symbol Device:L
- removed R801, R802: 100k, Resistor_SMD:R_0402_1005Metric, symbol Device:R
- removed R803: 22.1k, Resistor_SMD:R_0402_1005Metric, symbol Device:R
- removed U803: SY8883DFC, Package_DFN_QFN:DFN-8-1EP_2x2mm_P0.5mm_EP0.9x1.6mm, symbol MyLibrary:SY8883DFC
- added F301: 2A, Fuse:Fuse_1812_4532Metric, symbol Device:Fuse
Connections:
- net USBu_DN is gone; now on net USB_DN: U301.15 (DMU)
- net USBu_DP is gone; now on net USB_DP: U301.16 (DPU)
- net VBUS: now also F301.2; no longer C301.1, U301.18 (VBUSM), U301.20 (VDD5)
- new net +5V: C301.1, F301.1, U301.18 (VBUSM), U301.20 (VDD5)
Other:
- note removed: "DC-DC 3.3V"
- title: STM32 USB Audio Interface - USB and Power Supply -> STM32 USB Audio Interface - USB
- moved on the sheet: C301, C302, C303, C304, C314, C315, D301, D302, D303, D304, D305, D306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
