File: STM32-USB-Audio-Board/Schematics/mcu_daplink_ch32v305.kicad_sch (KiCad schematic)
At the start: 27 parts, among them J701 USB_B_Micro, J702 Conn_01x04, J703 Conn_01x05, SW701 SW_Push, SW702 SW_Push, SW703 SW_Push, U701 CH32V305RBT6, Y301 8MHz, Y701 32.768kHz

Commit message: Cleanup
Parts:
- removed R305: 0R, Resistor_SMD:R_0402_1005Metric, symbol Device:R
- J702: footprint (none) -> Connector_PinHeader_2.54mm:PinHeader_1x04_P2.54mm_Vertical
- J703: footprint (none) -> Connector_PinHeader_2.54mm:PinHeader_1x05_P2.54mm_Vertical
- U701: footprint Package_QFP:LQFP-48_7x7mm_P0.5mm -> Package_QFP:LQFP-64_10x10mm_P0.5mm
Connections:
- net +3.3V: now also SW701.1; no longer R701.1
- net GND: now also R701.2; no longer C311.2, SW701.2, U701.60 (BOOT0)
- net at U701.6 (OSC_OUT/PD1): now also C315.2, Y301.1
- new net BOOT0: C311.2, R701.1, SW701.2, U701.60 (BOOT0)
Changed lines of the file:
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@@
     (stroke (width 0) (type default))
   )
-  (wire (pts (xy 236.22 55.88) (xy 236.22 71.12))
+  (wire (pts (xy 236.22 55.88) (xy 236.22 59.69))
     (stroke (width 0) (type default))
   )
@@
     (stroke (width 0) (type default))
   )
-  (wire (pts (xy 105.41 139.7) (xy 127 139.7))
+  (wire (pts (xy 86.36 139.7) (xy 127 139.7))
     (stroke (width 0) (type default))
   )
@@
     (stroke (width 0) (type default))
   )
-  (wire (pts (xy 236.22 41.91) (xy 236.22 43.18))
-    (stroke (width 0) (type default))
-  )
-  (wire (pts (xy 236.22 33.02) (xy 236.22 34.29))
+  (wire (pts (xy 236.22 33.02) (xy 236.22 43.18))
     (stroke (width 0) (type default))
   )
@@
     (stroke (width 0) (type default))
   )
-  (wire (pts (xy 86.36 139.7) (xy 97.79 139.7))
-    (stroke (width 0) (type default))
-  )
   (wire (pts (xy 83.82 53.34) (xy 96.52 53.34))
     (stroke (width 0) (type default))
   )
   (wire (pts (xy 63.5 114.3) (xy 63.5 111.76))
+    (stroke (width 0) (type default))
+  )
+  (wire (pts (xy 236.22 67.31) (xy 236.22 71.12))
     (stroke (width 0) (type default))
   )
@@
       (effects (font (size 1.27 1.27)))
     )
-    (property "Footprint" "Package_QFP:LQFP-48_7x7mm_P0.5mm" (at 129.54 55.88 0)
+    (property "Footprint" "Package_QFP:LQFP-64_10x10mm_P0.5mm" (at 129.54 55.88 0)
       (effects (font (size 1.27 1.27)) hide)
     )
@@
     )
   )
-  (symbol (lib_id "Device:R") (at 101.6 139.7 90) (unit 1)
-    (in_bom yes) (on_board yes) (dnp no)
-    (property "Reference" "R305" (at 101.6 137.16 90)
-      (effects (font (size 1.27 1.27)))
-    )
-    (property "Value" "0R" (at 101.6 139.7 90)
-      (effects (font (size 1.27 1.27)))
-    )
-    (property "Footprint" "Resistor_SMD:R_0402_1005Metric" (at 101.6 141.478 90)
-      (effects (font (size 1.27 1.27)) hide)
-    )
-    (property "Datasheet" "~" (at 101.6 139.7 0)
-      (effects (font (size 1.27 1.27)) hide)
-    )
-    (pin "1")
-    (pin "2")
-    (instances
-      (project "Quad_RAK3172_Board"
-        (path "/07819ddb-8589-49ca-8cb1-e5fd69494837/ceadba99-10e5-4d21-a45c-0b114067dd5b"
-          (reference "R305") (unit 1)
-        )
-      )
-      (project "STM32-USB-Audio-Board"
-        (path "/b58c5c23-bc0f-41f0-a4fc-93f4cd916b6e/d07c0e8c-6a5b-4f18-bb65-05a2c61616e0"
-          (reference "R205") (unit 1)
-        )
-        (path "/b58c5c23-bc0f-41f0-a4fc-93f4cd916b6e/98639fa2-3e30-4103-8d18-092f7c1f3e80"
-          (reference "R704") (unit 1)
-        )
-      )
-    )
-  )
   (symbol (lib_id "power:GND") (at 109.22 66.04 0) (unit 1)
     (in_bom yes) (on_board yes) (dnp no)
@@
         (path "/b58c5c23-bc0f-41f0-a4fc-93f4cd916b6e/98639fa2-3e30-4103-8d18-092f7c1f3e80"
           (reference "#PWR0715") (unit 1)
-        )
-      )
-    )
-  )
-  (symbol (lib_id "Device:R") (at 236.22 38.1 0) (unit 1)
-    (in_bom yes) (on_board yes) (dnp no) (fields_autoplaced)
-    (property "Reference" "R701" (at 238.76 37.465 0)
-      (effects (font (size 1.27 1.27)) (justify left))
-    )
-    (property "Value" "10k" (at 238.76 40.005 0)
-      (effects (font (size 1.27 1.27)) (justify left))
-    )
-    (property "Footprint" "Resistor_SMD:R_0402_1005Metric" (at 234.442 38.1 90)
-      (effects (font (size 1.27 1.27)) hide)
-    )
-    (property "Datasheet" "~" (at 236.22 38.1 0)
-      (effects (font (size 1.27 1.27)) hide)
-    )
-    (pin "1")
-    (pin "2")
-    (instances
-      (project "STM32-USB-Audio-Board"
-        (path "/b58c5c23-bc0f-41f0-a4fc-93f4cd916b6e/98639fa2-3e30-4103-8d18-092f7c1f3e80"
-          (reference "R701") (unit 1)
         )
       )
@@
       (effects (font (size 1.27 1.27)) (justify left))
     )
-    (property "Footprint" "" (at 226.06 129.54 0)
+    (property "Footprint" "Connector_PinHeader_2.54mm:PinHeader_1x05_P2.54mm_Vertical" (at 226.06 129.54 0)
       (effects (font (size 1.27 1.27)) hide)
     )
@@
     )
   )
+  (symbol (lib_id "Device:R") (at 236.22 63.5 0) (unit 1)
+    (in_bom yes) (on_board yes) (dnp no) (fields_autoplaced)
+    (property "Reference" "R701" (at 238.76 62.865 0)
+      (effects (font (size 1.27 1.27)) (justify left))
+    )
+    (property "Value" "10k" (at 238.76 65.405 0)
+      (effects (font (size 1.27 1.27)) (justify left))
+    )
+    (property "Footprint" "Resistor_SMD:R_0402_1005Metric" (at 234.442 63.5 90)
+      (effects (font (size 1.27 1.27)) hide)
+    )
+    (property "Datasheet" "~" (at 236.22 63.5 0)
+      (effects (font (size 1.27 1.27)) hide)
+    )
+    (pin "1")
+    (pin "2")
+    (instances
+      (project "STM32-USB-Audio-Board"
+        (path "/b58c5c23-bc0f-41f0-a4fc-93f4cd916b6e/98639fa2-3e30-4103-8d18-092f7c1f3e80"
+          (reference "R701") (unit 1)
+        )
+      )
+    )
+  )
   (symbol (lib_id "Connector_Generic:Conn_01x04") (at 256.54 127 0) (unit 1)
     (in_bom yes) (on_board yes) (dnp no) (fields_autoplaced)
@@
       (effects (font (size 1.27 1.27)) (justify left))
     )
-    (property "Footprint" "" (at 256.54 127 0)
-      (effects (font (size 1.27 1.27)) hide)
-    )
+    (property "Footprint" "Connector_PinHeader_2.54mm:PinHeader_1x04_P2.54mm_Vertical" (at 256.54 127 0)
+      (effects (font (size 1.27 1.27)) hide)
+    )
